File: Electronique/Rolling_Base/PCB/power_part.sch (KiCad schematic (older format))
At the start: 29 parts, among them J3 FAN, U11 B_Plug_5mm, U12 B_Plug_5mm, U13 LM317_SOT223, U14 LM317_SOT223

Commit message: Utilisation de chemin relatif au projet pour les librairies
Connections:
- net labels added: +3V3
- net labels removed: +3.3V
Changed lines of the file:
@@
 EESchema Schematic File Version 4
-LIBS:Motor_Card-cache
 EELAYER 26 0
 EELAYER END
@@
 $EndDescr
 $Comp
-L Motor_Card-rescue:+3.3V- #PWR?
-U 1 1 5962E5EC
-P 10425 2500
-AR Path="/5962E5EC" Ref="#PWR?"  Part="1"
-AR Path="/59613F6F/5962E5EC" Ref="#PWR061"  Part="1"
-F 0 "#PWR061" H 10425 2350 50  0001 C CNN
-F 1 "+3.3V" H 10425 2640 50  0000 C CNN
-F 2 "" H 10425 2500 50  0001 C CNN
-F 3 "" H 10425 2500 50  0001 C CNN
-	1    10425 2500
-	1    0    0    -1
-$EndComp
-$Comp
 L 2:B_Plug_5mm U11
 U 1 1 5962E6CD
@@
 L Regulator_Linear:LM317_3PinPackage U14
 U 1 1 5962EF34
-P 9625 2550
-F 0 "U14" H 9625 2550 50  0000 C CNN
-F 1 "LM317_SOT223" H 9675 2300 50  0000 L CNN
-F 2 "TO_SOT_Packages_SMD:SOT-223-3Lead_TabPin2" H 9625 2550 50  0001 C CNN
-F 3 "" H 9625 2550 50  0001 C CNN
-	1    9625 2550
+P 9600 2550
+F 0 "U14" H 9600 2550 50  0000 C CNN
+F 1 "LM317_SOT223" H 9650 2300 50  0000 L CNN
+F 2 "TO_SOT_Packages_SMD:SOT-223-3Lead_TabPin2" H 9600 2550 50  0001 C CNN
+F 3 "" H 9600 2550 50  0001 C CNN
+	1    9600 2550
 	1    0    0    -1
 $EndComp
@@
 	7900 2450 7900 2550
 Wire Wire Line
-	9025 2500 9025 2550
-Wire Wire Line
-	10425 2500 10425 2550
+	9000 2500 9000 2550
+Wire Wire Line
+	10400 2500 10400 2550
 $Comp
 L Device:R R7
@@
 L Device:R R10
 U 1 1 5962F32D
-P 9625 3400
-F 0 "R10" V 9705 3400 50  0000 C CNN
-F 1 "370" V 9625 3400 50  0000 C CNN
-F 2 "Resistor_SMD:R_1206_3216Metric_Pad1.42x1.75mm_HandSolder" V 9555 3400 50  0001 C CNN
-F 3 "" H 9625 3400 50  0001 C CNN
-	1    9625 3400
+P 9600 3400
+F 0 "R10" V 9680 3400 50  0000 C CNN
+F 1 "370" V 9600 3400 50  0000 C CNN
+F 2 "Resistor_SMD:R_1206_3216Metric_Pad1.42x1.75mm_HandSolder" V 9530 3400 50  0001 C CNN
+F 3 "" H 9600 3400 50  0001 C CNN
+	1    9600 3400
 	-1   0    0    1
 $EndComp
@@
 L Device:R R11
 U 1 1 5962F372
-P 9975 3200
-F 0 "R11" V 10055 3200 50  0000 C CNN
-F 1 "220" V 9975 3200 50  0000 C CNN
-F 2 "Resistor_SMD:R_1206_3216Metric_Pad1.42x1.75mm_HandSolder" V 9905 3200 50  0001 C CNN
-F 3 "" H 9975 3200 50  0001 C CNN
-	1    9975 3200
+P 9950 3200
+F 0 "R11" V 10030 3200 50  0000 C CNN
+F 1 "220" V 9950 3200 50  0000 C CNN
+F 2 "Resistor_SMD:R_1206_3216Metric_Pad1.42x1.75mm_HandSolder" V 9880 3200 50  0001 C CNN
+F 3 "" H 9950 3200 50  0001 C CNN
+	1    9950 3200
 	0    1    1    0
 $EndComp
@@
 L power:GND #PWR060
 U 1 1 5962F3F1
-P 9625 3650
-F 0 "#PWR060" H 9625 3400 50  0001 C CNN
-F 1 "GND" H 9625 3500 50  0000 C CNN
-F 2 "" H 9625 3650 50  0001 C CNN
-F 3 "" H 9625 3650 50  0001 C CNN
-	1    9625 3650
+P 9600 3650
+F 0 "#PWR060" H 9600 3400 50  0001 C CNN
+F 1 "GND" H 9600 3500 50  0000 C CNN
+F 2 "" H 9600 3650 50  0001 C CNN
+F 3 "" H 9600 3650 50  0001 C CNN
+	1    9600 3650
 	1    0    0    -1
 $EndComp
@@
 	7650 3150 7650 2550
 Wire Wire Line
-	9625 3250 9625 3200
-Wire Wire Line
-	9625 3650 9625 3550
-Wire Wire Line
-	9825 3200 9625 3200
-Connection ~ 9625 3200
-Wire Wire Line
-	10125 3200 10275 3200
-Wire Wire Line
-	10275 3200 10275 2550
-Connection ~ 10275 2550
+	9600 3250 9600 3200
+Wire Wire Line
+	9600 3650 9600 3550
+Wire Wire Line
+	9800 3200 9600 3200
+Connection ~ 9600 3200
+Wire Wire Line
+	10100 3200 10250 3200
+Wire Wire Line
+	10250 3200 10250 2550
+Connection ~ 10250 2550
 $Comp
 L Device:R R6
@@
 L Device:R R12
 U 1 1 596302DA
-P 10625 2550
-F 0 "R12" V 10705 2550 50  0000 C CNN
-F 1 "470" V 10625 2550 50  0000 C CNN
-F 2 "Resistor_SMD:R_1206_3216Metric_Pad1.42x1.75mm_HandSolder" V 10555 2550 50  0001 C CNN
-F 3 "" H 10625 2550 50  0001 C CNN
-	1    10625 2550
+P 10600 2550
+F 0 "R12" V 10680 2550 50  0000 C CNN
+F 1 "470" V 10600 2550 50  0000 C CNN
+F 2 "Resistor_SMD:R_1206_3216Metric_Pad1.42x1.75mm_HandSolder" V 10530 2550 50  0001 C CNN
+F 3 "" H 10600 2550 50  0001 C CNN
+	1    10600 2550
 	0    1    1    0
 $EndComp
@@
 L Device:LED_ALT D11
 U 1 1 59630393
-P 10825 2800
-F 0 "D11" H 10825 2900 50  0000 C CNN
-F 1 "LED_3.3V" H 10825 2650 50  0000 C CNN
-F 2 "Diodes_SMD:D_SMA-SMB_Universal_Handsoldering" H 10825 2800 50  0001 C CNN
-F 3 "" H 10825 2800 50  0001 C CNN
-	1    10825 2800
+P 10800 2800
+F 0 "D11" H 10800 2900 50  0000 C CNN
+F 1 "LED_3.3V" H 10800 2650 50  0000 C CNN
+F 2 "Diodes_SMD:D_SMA-SMB_Universal_Handsoldering" H 10800 2800 50  0001 C CNN
+F 3 "" H 10800 2800 50  0001 C CNN
+	1    10800 2800
 	0    -1   -1   0
 $EndComp
@@
 L power:GND #PWR063
 U 1 1 596306A0
-P 10825 3150
-F 0 "#PWR063" H 10825 2900 50  0001 C CNN
-F 1 "GND" H 10825 3000 50  0000 C CNN
-F 2 "" H 10825 3150 50  0001 C CNN
-F 3 "" H 10825 3150 50  0001 C CNN
-	1    10825 3150
-	1    0    0    -1
-$EndComp
-Connection ~ 10425 2550
-Wire Wire Line
-	10775 2550 10825 2550
-Wire Wire Line
-	10825 2550 10825 2650
-Wire Wire Line
-	10825 2950 10825 3150
+P 10800 3150
+F 0 "#PWR063" H 10800 2900 50  0001 C CNN
+F 1 "GND" H 10800 3000 50  0000 C CNN
+F 2 "" H 10800 3150 50  0001 C CNN
+F 3 "" H 10800 3150 50  0001 C CNN
+	1    10800 3150
+	1    0    0    -1
+$EndComp
+Connection ~ 10400 2550
+Wire Wire Line
+	10750 2550 10800 2550
+Wire Wire Line
+	10800 2550 10800 2650
+Wire Wire Line
+	10800 2950 10800 3150
 Connection ~ 7900 2550
 Wire Wire Line
@@
 L Device:C C8
 U 1 1 5962624A
-P 10425 2900
-F 0 "C8" H 10450 3000 50  0000 L CNN
-F 1 "10u" H 10450 2800 50  0000 L CNN
-F 2 "Capacitor_THT:CP_Radial_D8.0mm_P3.50mm" H 10463 2750 50  0001 C CNN
-F 3 "" H 10425 2900 50  0001 C CNN
-	1    10425 2900
+P 10400 2900
+F 0 "C8" H 10425 3000 50  0000 L CNN
+F 1 "10u" H 10425 2800 50  0000 L CNN
+F 2 "Capacitor_THT:CP_Radial_D8.0mm_P3.50mm" H 10438 2750 50  0001 C CNN
+F 3 "" H 10400 2900 50  0001 C CNN
+	1    10400 2900
 	1    0    0    -1
 $EndComp
@@
 L power:GND #PWR062
 U 1 1 5962633A
-P 10425 3400
-F 0 "#PWR062" H 10425 3150 50  0001 C CNN
-F 1 "GND" H 10425 3250 50  0000 C CNN
-F 2 "" H 10425 3400 50  0001 C CNN
-F 3 "" H 10425 3400 50  0001 C CNN
-	1    10425 3400
+P 10400 3400
+F 0 "#PWR062" H 10400 3150 50  0001 C CNN
+F 1 "GND" H 10400 3250 50  0000 C CNN
+F 2 "" H 10400 3400 50  0001 C CNN
+F 3 "" H 10400 3400 50  0001 C CNN
+	1    10400 3400
 	1    0    0    -1
 $EndComp
@@
 	7900 3300 7900 3100
 Wire Wire Line
-	10425 3050 10425 3400
+	10400 3050 10400 3400
 $Comp
 L Device:C C5
@@
 	2450 2400 2450 2450
 Wire Wire Line
-	10275 2550 10425 2550
-Wire Wire Line
-	10425 2550 10425 2750
-Wire Wire Line
-	10425 2550 10475 2550
+	10250 2550 10400 2550
+Wire Wire Line
+	10400 2550 10400 2750
+Wire Wire Line
+	10400 2550 10450 2550
 Wire Wire Line
 	7900 2550 7900 2800
@@
 	7000 2850 7000 3150
 Wire Wire Line
-	9925 2550 10275 2550
-Wire Wire Line
-	9025 2550 9325 2550
-Wire Wire Line
-	9625 2850 9625 3200
+	9900 2550 10250 2550
+Wire Wire Line
+	9000 2550 9300 2550
+Wire Wire Line
+	9600 2850 9600 3200
 Wire Wire Line
 	3275 2100 3575 2100
@@
 L power:+10V #PWR058
 U 1 1 5C206EB6
-P 9025 2500
-F 0 "#PWR058" H 9025 2350 50  0001 C CNN
-F 1 "+10V" H 9040 2673 50  0000 C CNN
-F 2 "" H 9025 2500 50  0001 C CNN
-F 3 "" H 9025 2500 50  0001 C CNN
-	1    9025 2500
+P 9000 2500
+F 0 "#PWR058" H 9000 2350 50  0001 C CNN
+F 1 "+10V" H 9015 2673 50  0000 C CNN
+F 2 "" H 9000 2500 50  0001 C CNN
+F 3 "" H 9000 2500 50  0001 C CNN
+	1    9000 2500
 	1    0    0    -1
 $EndComp
@@
 L Device:C Cin_2
 U 1 1 5C24DAB9
-P 9025 2700
-F 0 "Cin_2" H 8825 2800 50  0000 L CNN
-F 1 "0,1u" H 8775 2600 50  0000 L CNN
-F 2 "Capacitor_SMD:C_1206_3216Metric_Pad1.42x1.75mm_HandSolder" H 9063 2550 50  0001 C CNN
-F 3 "~" H 9025 2700 50  0001 C CNN
-	1    9025 2700
+P 9000 2700
+F 0 "Cin_2" H 8800 2800 50  0000 L CNN
+F 1 "0,1u" H 8750 2600 50  0000 L CNN
+F 2 "Capacitor_SMD:C_1206_3216Metric_Pad1.42x1.75mm_HandSolder" H 9038 2550 50  0001 C CNN
+F 3 "~" H 9000 2700 50  0001 C CNN
+	1    9000 2700
 	1    0    0    -1
 $EndComp
@@
 L power:GND #PWR059
 U 1 1 5C24DAC0
-P 9025 2850
-F 0 "#PWR059" H 9025 2600 50  0001 C CNN
-F 1 "GND" H 9025 2700 50  0000 C CNN
-F 2 "" H 9025 2850 50  0001 C CNN
-F 3 "" H 9025 2850 50  0001 C CNN
-	1    9025 2850
+P 9000 2850
+F 0 "#PWR059" H 9000 2600 50  0001 C CNN
+F 1 "GND" H 9000 2700 50  0000 C CNN
+F 2 "" H 9000 2850 50  0001 C CNN
+F 3 "" H 9000 2850 50  0001 C CNN
+	1    9000 2850
 	1    0    0    -1
 $EndComp
@@
 Wire Wire Line
 	2500 3550 2500 3575
+$Comp
+L power:+3V3 #PWR?
+U 1 1 5C54A8A0
+P 10400 2500
+F 0 "#PWR?" H 10400 2350 50  0001 C CNN
+F 1 "+3V3" H 10415 2673 50  0000 C CNN
+F 2 "" H 10400 2500 50  0001 C CNN
+F 3 "" H 10400 2500 50  0001 C CNN
+	1    10400 2500
+	1    0    0    -1
+$EndComp
+Connection ~ 9000 2550
 $EndSCHEMATC
