File: Electronique/Rolling_Base/PCB/power_part.sch (KiCad schematic (older format))
At the start: 29 parts, among them J3 FAN, U11 B_Plug_5mm, U12 B_Plug_5mm, U13 LM317_SOT223, U14 LM317_SOT223

Commit message: Final Rolling Base Card
Parts:
- C3, C4, C7, C8: RS-1 (none) -> Plein au Club
- C5, C6, Cin_1, Cin_2: RS-1 (none) -> https://fr.farnell.com/vishay/vj1206y104kxxpw1bc/condensate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
- D10, D11, D8, D9: footprint Diodes_SMD:D_SMA-SMB_Universal_Handsoldering -> LED_SMD:LED_1206_3216Metric; RS-1 (none) -> https://fr.farnell.com/kingbright/kpt-1608lvvbc-d/led-bleue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
- D6, D7: footprint Diodes_SMD:D_SMA_Handsoldering -> Diode_SMD:D_SMA_Handsoldering; RS-1 (none) -> https://fr.farnell.com/taiwan-semiconductor/rs1al/diode-fas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
- F1: value Fuse -> Fuse_Puiss; RS-1 (none) -> https://fr.farnell.com/multicomp/mccfb1206ttt-6/fusible-6a-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
- F2: value Fuse -> Fuse_Num; RS-1 (none) -> https://fr.farnell.com/multicomp/mccfb1206ttt-4/fusible-4a-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
- J3: footprint Connectors_Molex:Molex_KK-6410-02_02x2.54mm_Straight -> Connector_Molex:Molex_KK-254_AE-6410-02A_1x02_P2.54mm_Vertical; RS-1 (none) -> https://fr.rs-online.com/web/p/embases-de-circuit-imprime/1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; RS-2 (none) -> https://fr.rs-online.com/web/p/boitier-pour-connecteur-ci/2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
- R10: RS-1 (none) -> https://fr.farnell.com/panasonic-electronic-components/erj8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
- R11: RS-1 (none) -> https://fr.farnell.com/multicomp/mcwr12x2200ftl/res-couche-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
- R12, R9: RS-1 (none) -> https://fr.farnell.com/multicomp/mchp06w2f4700t5e/res-couch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
- R5, R6: RS-1 (none) -> https://fr.farnell.com/multicomp/mcwr12x2001ftl/res-couche-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
- R7: RS-1 (none) -> https://fr.farnell.com/vishay/crcw1206820rfkea/res-couche-e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
- R8: RS-1 (none) -> https://fr.farnell.com/tt-electronics-welwyn/wcr1206-270rfi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
- U11, U12: footprint B plug:B plug 5mm -> B plug:Bplug-5mm; RS-1 (none) -> Plein au club
- U13, U14: footprint TO_SOT_Packages_SMD:SOT-223-3Lead_TabPin2 -> Package_TO_SOT_SMD:SOT-223-3_TabPin2; RS-1 (none) -> https://fr.farnell.com/texas-instruments/lm317aemp-nopb/reg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
