File: Electronique/Rolling_Base/PCB/Motor_Card.sch (KiCad schematic (older format))
At the start: 4 parts, among them U1 Trou-3, U2 Trou-3, U3 Trou-3, U4 Trou-3

Commit message: Final Rolling Base Card
Parts:
- U1, U2, U3, U4: RS-1 (none) -> C'est un trou de perçage
Changed lines of the file:
@@
 F 2 "maxon:Trou-3" H 2000 4150 60  0001 C CNN
 F 3 "" H 2000 4150 60  0000 C CNN
+F 4 "C'est un trou de perçage" H 0   0   50  0001 C CNN "RS-1"
 	1    2000 4150
 	1    0    0    -1
@@
 F 2 "maxon:Trou-3" H 2000 4400 60  0001 C CNN
 F 3 "" H 2000 4400 60  0000 C CNN
+F 4 "C'est un trou de perçage" H 0   0   50  0001 C CNN "RS-1"
 	1    2000 4400
 	1    0    0    -1
@@
 F 2 "maxon:Trou-3" H 2000 4700 60  0001 C CNN
 F 3 "" H 2000 4700 60  0000 C CNN
+F 4 "C'est un trou de perçage" H 0   0   50  0001 C CNN "RS-1"
 	1    2000 4700
 	1    0    0    -1
@@
 F 2 "maxon:Trou-3" H 2000 5000 60  0001 C CNN
 F 3 "" H 2000 5000 60  0000 C CNN
+F 4 "C'est un trou de perçage" H 0   0   50  0001 C CNN "RS-1"
 	1    2000 5000
 	1    0    0    -1
