File: Electronique/Rolling_Base/PCB/motor_part.sch (KiCad schematic (older format))
At the start: 42 parts, among them K1 Maxon-200142, K2 Maxon-200142, U5 L6235D, U6 L6235D

Commit message: Final Rolling Base Card
Parts:
- removed RH1, RH2, RH3, RH4, RH5, RH6: 10k, Resistor_SMD:R_1206_3216Metric_Pad1.42x1.75mm_HandSolder, symbol Device:R
- Cboot1, Cboot2: RS-1 (none) -> https://fr.farnell.com/yageo/cc1206krx7r8bb224/cond-0-22-f-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
- Cen1, Cen2: RS-1 (none) -> https://fr.farnell.com/multicomp/mc1206b562k500ct/cond-5600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
- Coff1, Coff2: RS-1 (none) -> https://fr.farnell.com/vishay/vj1206y102kxxpw1bc/cond-1000p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
- Cp1, Cp2, Cpul1, Cpul2, Cref1, Cref2: RS-1 (none) -> https://fr.farnell.com/vishay/vj1206y103kxjcw1bc/cond-0-01-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
- D1, D2, D3, D4: footprint Diodes_THT:D_DO-35_SOD27_P10.16mm_Horizontal -> Diode_THT:D_DO-35_SOD27_P10.16mm_Horizontal; RS-1 (none) -> https://fr.farnell.com/vishay/1n4148tr/diode-de-redressemen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
- K1, K2: RS-1 (none) -> https://eu.mouser.com/ProductDetail/Molex/52610-1133?qs=rw2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
- Ren1, Ren2: RS-1 (none) -> https://fr.farnell.com/te-connectivity/crgcq1206j100k/resi-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
- Roff1, Roff2: RS-1 (none) -> https://fr.farnell.com/te-connectivity/crgcq1206j33k/res-ae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
- Rp1, Rp2: RS-1 (none) -> https://fr.farnell.com/multicomp/mcwr12x1000ftl/resistance-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
- Rpul1, Rpul2: RS-1 (none) -> https://fr.farnell.com/multicomp/mcsr12x4702ftl/res-ceramiq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
- Rref1, Rref3: RS-1 (none) -> https://fr.farnell.com/te-connectivity/crgcq1206f1k2/res-ae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
- Rref2, Rref4: RS-1 (none) -> https://fr.farnell.com/te-connectivity/crgcq1206j220r/resi-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
- Rsense1, Rsense2: RS-1 (none) -> https://fr.farnell.com/bourns/crl1206-jw-r300elf/res-couche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
- Rtacho1, Rtacho2: RS-1 (none) -> https://fr.farnell.com/te-connectivity/crgcq1206j1k0/res-ae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
- U5, U6: footprint Housings_SOIC:SOIC-24W_7.5x15.4mm_Pitch1.27mm -> Package_SO:SOIC-24W_7.5x15.4mm_P1.27mm; RS-1 (none) -> Contact ST
Connections:
- wire segments 162 -> 146
Other:
- note added: "Résistances de Pull-Up déjà présentes dans le moteur"
