File: Electronique/Rolling_Base/PCB/uC.sch (KiCad schematic (older format))
At the start: 24 parts, among them J1 CONN_SERIAL, J2 swdio, P1 CONN_I2C, P2 CONN_FREE, U10 txb0108, U15 txb0108, U7 74HC00, U8 stm32f303k8t6, U9 txb0108

Commit message: Final Rolling Base Card
Parts:
- removed C10, C9: 0,1u, Capacitor_SMD:C_1206_3216Metric_Pad1.42x1.75mm_HandSolder, symbol Device:C
- removed U15: txb0108, Package_SO:TSSOP-20_4.4x6.5mm_P0.65mm, symbol stm32f042k6tx:txb0108
- C1, C13, C14, C15, C2: RS-1 (none) -> https://fr.farnell.com/vishay/vj1206y104kxxpw1bc/condensate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
- C11, C12: RS-1 (none) -> https://fr.farnell.com/walsin/1206b104k250ct/cond-0-1-f-25v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
- D5: footprint Diodes_SMD:D_SMA-SMB_Universal_Handsoldering -> LED_SMD:LED_1206_3216Metric; RS-1 (none) -> https://fr.farnell.com/kingbright/kpt-1608lvvbc-d/led-bleue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
- J1, P1, P2: footprint Connectors_Molex:Molex_KK-6410-02_02x2.54mm_Straight -> Connector_Molex:Molex_KK-254_1x02_P2.54mm_Horizontal; RS-1 (none) -> https://fr.rs-online.com/web/p/embases-de-circuit-imprime/1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; RS-2 (none) -> https://fr.rs-online.com/web/p/boitier-pour-connecteur-ci/2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
- J2: footprint Pin_Headers:Pin_Header_Straight_1x04_Pitch2.54mm -> Connector_Molex:Molex_KK-254_AE-6410-04A_1x04_P2.54mm_Vertical; RS-1 (none) -> https://fr.rs-online.com/web/p/embases-de-circuit-imprime/4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; RS-2 (none) -> https://fr.rs-online.com/web/p/boitier-pour-connecteur-ci/2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
- JP1: footprint Pin_Headers:Pin_Header_Straight_1x03_Pitch2.54mm -> Connector_PinHeader_2.54mm:PinHeader_1x03_P2.54mm_Vertical; RS-1 (none) -> Plein au club; RS-2 (none) -> https://fr.rs-online.com/web/p/products/467598/
- R1, R2, R3: RS-1 (none) -> https://fr.farnell.com/tt-electronics-welwyn/wcr1206-10kfi/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
- R4: RS-1 (none) -> https://fr.farnell.com/multicomp/mchp06w2f4700t5e/res-couch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
- U10: renamed from U9; RS-1 (none) -> https://fr.farnell.com/texas-instruments/txb0108pwr/ic-tran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
- U10, U9: RS-1 (none) -> https://fr.farnell.com/texas-instruments/txb0108pwr/ic-tran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
- U7: RS-1 (none) -> https://fr.rs-online.com/web/p/portes-logiques/6631865/
- U8: footprint Housings_QFP:LQFP-32_7x7mm_Pitch0.8mm -> Package_QFP:LQFP-32_7x7mm_P0.8mm; RS-1 (none) -> Contact ST
Connections:
- wire segments 100 -> 89
Other:
- note removed: "Conversion des tensions pour les connecteurs de sortie\n"
