File: Electronique/Power_Circuit/Power_Circuit.sch (KiCad schematic (older format))
At the start: 45 parts, among them U1 B_Plug_5mm, U10 B_Plug_5mm, U11 B_Plug_5mm, U12 B_Plug_5mm, U13 B_Plug_5mm, U14 B_Plug_5mm, U15 DSN2596, U16 DSN2596, U17 B_Plug_5mm, U18 B_Plug_5mm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

Commit message: Circuit adjustement
Parts:
- removed D1: LED, LED_SMD:LED_1206_3216Metric_Pad1.42x1.75mm_HandSolder, symbol Device:LED
- removed R1: R, Resistor_SMD:R_1206_3216Metric_Pad1.42x1.75mm_HandSolder, symbol Device:R
- removed U1, U2: B_Plug_5mm, dsn2596:B plug 5mm, symbol 2:B_Plug_5mm
- added D6, D7: LED, LED_SMD:LED_1206_3216Metric_Pad1.42x1.75mm_HandSolder, symbol Device:LED
- added F4: Fuse, Fuse:Fuse_1206_3216Metric_Pad1.42x1.75mm_HandSolder, symbol Device:Fuse
- added H8: MountingHole_Pad, Connector_PinHeader_1.00mm:PinHeader_1x01_P1.00mm_Horizontal, symbol Mechanical:MountingHole_Pad
- added R5, R6: R, Resistor_SMD:R_1206_3216Metric_Pad1.42x1.75mm_HandSolder, symbol Device:R
- added U19: DSN2596, dsn2596:DSN2596, symbol dsn2596:DSN2596
- added U20: B_Plug_5mm, dsn2596:B plug 5mm, symbol 2:B_Plug_5mm
- gave numbers to parts that had none: 9
Connections:
- net Battery is gone; now on net Raspberr_5V: H1.1
- net 12V: now also U19.1 (IN+)
- net 18V: now also C1.1, R5.1
- net GND: now also D6.1 (K), D7.1 (K), U19.2 (IN-), U19.3 (OUT-), U20.2
- net Logical_10V: now also R2.1
- net Motor1_12V: now also F5.1, U17.1; no longer F5.2, U15.4 (OUT+)
- net Motor2_12V: now also F6.1, U18.1; no longer F6.2, U16.4 (OUT+)
- net at F3.2, U5.4 (OUT+): no longer R2.1
- net at F1.2, U3.1: no longer C1.1
- net Raspberr_5V: now reaches C2.1, F2.1, R1.2, U1.1
- new net: F5.2, U15.4 (OUT+)
- new net: F6.2, U16.4 (OUT+)
- new net: D6.2 (A), R5.2
- new net: F4.2, U19.4 (OUT+)
- new net: D7.2 (A), R6.2
- new net MotorExt_12V: F4.1, H8.1, R6.1, U20.1
Other:
- moved on the sheet: C1, C2, D1, D3, D4, D5, F1, F2, F3, F5, F6, H5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
